Commit message: Add files via upload

File: urdf/interaction_base.xacro (robot description, xacro)
@@ -192,121 +192,3 @@
     </actuator>
   </transmission>
-  <!-- arm -->
-  <joint type="fixed" name="arm_base_joint">
-    <parent link="base_link"/>
-    <child link="arm_base"/>
-    <origin xyz="0.055 0.0 1.06" rpy="0 0 0"/>
-  </joint>
-  <link name="arm_base">
-    <visual name="visual">
-      <origin xyz="0.0 0 0.0" rpy="0 0 0"/>
-      <geometry>
-	      <box size=".05 .07 .09"/>
-      </geometry>
-      <material name="orange"/>
-    </visual>
-  </link>
-  <joint type="revolute" name="arm_joint_0">
-    <parent link="arm_base"/>
-    <child link="arm_link_1"/>
-    <origin xyz="0.025 0.0 0.035" rpy="0 0 0"/>
-    <axis xyz="1 0 0" rpy="0 0 0"/>
-    <limit effort="100" velocity="100.0"  lower="-1.5" upper="1.5" />
-  </joint>
-  <link name="arm_link_1">
-    <visual name="visual">
-      <origin xyz="0.035 0 0.0" rpy="0 0 0"/>
-      <geometry>
-	      <box size="0.07 0.04 0.04"/>
-      </geometry>
-      <material name="orange"/>
-    </visual>
-  </link>
-  <joint type="revolute" name="arm_joint_1">
-    <parent link="arm_link_1"/>
-    <child link="arm_link_2"/>
-    <origin xyz="0.05 0.0 0.0" rpy="3.14 0 0"/>
-    <axis xyz="0 0 1" rpy="0 0 0"/>
-    <limit effort="100" velocity="100.0"  lower="-1.5" upper="1.5" />
-  </joint>
-   <link name="arm_link_2">
-    <visual name="visual">
-      <origin xyz="0.04 0 0" rpy="0 0 0"/>
-      <geometry>
-	      <box size="0.08 0.06 0.06"/>
-      </geometry>
-      <material name="orange"/>
-    </visual>
-  </link>
-  <joint type="revolute" name="arm_joint_2">
-    <parent link="arm_link_2"/>
-    <child link="arm_link_3"/>
-    <origin xyz="0.05 0.0 0.0" rpy="3.14 0.3 0"/>
-    <axis xyz="0 1 0" rpy="0 0 0"/>
-    <limit effort="100" velocity="100.0"  lower="-3.14" upper="0" />
-  </joint>
-  <link name="arm_link_3">
-    <visual name="visual">
-      <origin xyz="0.0 0. -0.13" rpy="0 0 0"/>
-      <geometry>
-	      <box size="0.05 0.05 0.28"/>
-      </geometry>
-      <material name="orange"/>
-    </visual>
-  </link>
-  <joint type="revolute" name="arm_joint_3">
-    <parent link="arm_link_3"/>
-    <child link="arm_link_4"/>
-    <origin xyz="0.0 0.0 -0.25" rpy="0 -3 0"/>
-    <axis xyz="0 1 0" rpy="0 0 0"/>
-    <limit effort="100" velocity="100.0"  lower="0" upper="3.14" />
-  </joint>
-  <link name="arm_link_4">
-    <collision>
-      <origin xyz="-0.05 0 -0.13" rpy="0 0 0"/>
-      <geometry>
-	      <box size="0.05 0.05 0.10"/>
-      </geometry>
-      <material name="orange"/>
-    </collision>
-    <visual name="visual">
-      <origin xyz="-0.05 0 -0.13" rpy="0 0 0"/>
-      <geometry>
-	      <box size="0.05 0.05 0.25"/>
-      </geometry>
-    <material name="orange"/>
-    </visual>
-  </link>
-  <joint type="revolute" name="arm_joint_4">
-    <parent link="arm_link_4"/>
-    <child link="arm_link_5"/>
-    <origin xyz="-0.045 0.0 -0.23" rpy="0 0 3.14"/>
-    <axis xyz="0 1 0" rpy="0 0 0"/>
-    <limit effort="100" velocity="100.0"  lower="-1.57" upper="1.57" />
-  </joint>
-  <link name="arm_link_5">
-    <visual name="visual">
-      <origin xyz="0.0 0 -0.03" rpy="0 0 0"/>
-      <geometry>
-	      <box size="0.05 0.05 0.08"/>
-      </geometry>
-      <material name="orange"/>
-    </visual>
-  </link>
-  <joint type="revolute" name="arm_joint_5">
-    <parent link="arm_link_5"/>
-    <child link="arm_link_6"/>
-    <origin xyz="0.0 0.0 -0.06" rpy="0 0 0"/>
-    <axis xyz="1 0 0" rpy="0 0 0"/>
-    <limit effort="100" velocity="100.0"  lower="-1.57" upper="1.57" />
-  </joint>
-  <link name="arm_link_6">
-    <visual name="visual">
-      <origin xyz="0.0 0 -0.04" rpy="0 0 0"/>
-      <geometry>
-	      <box size="0.05 0.03 0.03"/>
-      </geometry>
-      <material name="orange"/>
-    </visual>
-  </link>
 </robot>
