Commit message: add collision

File: urdf/interaction_robot.xacro (robot description, xacro)
@@ -200,4 +200,10 @@
   </joint>
   <link name="arm_base">
+    <collision>
+      <origin xyz="0.0 0 0.0" rpy="0 0 0"/>
+      <geometry>
+	      <box size=".05 .07 .09"/>
+      </geometry>
+    </collision>
     <visual name="visual">
       <origin xyz="0.0 0 0.0" rpy="0 0 0"/>
@@ -215,4 +221,10 @@
   </joint>
   <link name="arm_link_1">
+    <collision>
+      <origin xyz="0.035 0 0.0" rpy="0 0 0"/>
+      <geometry>
+	      <box size="0.07 0.04 0.04"/>
+      </geometry>
+    </collision>
     <visual name="visual">
       <origin xyz="0.035 0 0.0" rpy="0 0 0"/>
@@ -230,4 +242,10 @@
   </joint>
    <link name="arm_link_2">
+    <collision>
+      <origin xyz="0.04 0 0" rpy="0 0 0"/>
+      <geometry>
+	      <box size="0.08 0.06 0.06"/>
+      </geometry>
+    </collision>
     <visual name="visual">
       <origin xyz="0.04 0 0" rpy="0 0 0"/>
@@ -245,4 +263,10 @@
   </joint>
   <link name="arm_link_3">
+    <collision>
+      <origin xyz="0.0 0. -0.13" rpy="0 0 0"/>
+      <geometry>
+	      <box size="0.05 0.05 0.28"/>
+      </geometry>
+    </collision>
     <visual name="visual">
       <origin xyz="0.0 0. -0.13" rpy="0 0 0"/>
@@ -260,4 +284,10 @@
   </joint>
   <link name="arm_link_4">
+    <collision>
+      <origin xyz="0.05 0 -0.13" rpy="0 0 0"/>
+      <geometry>
+	      <box size="0.05 0.05 0.25"/>
+      </geometry>
+    </collision>
     <visual name="visual">
       <origin xyz="0.05 0 -0.13" rpy="0 0 0"/>
@@ -275,4 +305,10 @@
   </joint>
   <link name="arm_link_5">
+    <collision>
+      <origin xyz="0.0 0 -0.03" rpy="0 0 0"/>
+      <geometry>
+	      <box size="0.05 0.05 0.08"/>
+      </geometry>
+    </collision>
     <visual name="visual">
       <origin xyz="0.0 0 -0.03" rpy="0 0 0"/>
@@ -290,9 +326,15 @@
   </joint>
   <link name="arm_link_6">
-    <visual name="visual">
+    <collision>
       <origin xyz="0.0 0 -0.04" rpy="0 0 0"/>
       <geometry>
 	      <box size="0.05 0.03 0.05"/>
       </geometry>
+    </collision>
+    <visual name="visual">
+      <origin xyz="0.0 0 -0.04" rpy="0 0 0"/>
+      <geometry>
+	      <box size="0.05 0.03 0.05"/>
+      </geometry>
     </visual>
   </link>

Commit message: fix model

File: urdf/interaction_robot.xacro (robot description, xacro)
@@ -258,7 +258,7 @@
     <parent link="arm_link_3"/>
     <child link="arm_link_4"/>
-    <origin xyz="0.0 0.0 -0.25" rpy="0 -3 0"/>
+    <origin xyz="0.0 0.0 -0.25" rpy="0 -0.3 3.14"/>
     <axis xyz="0 1 0" rpy="0 0 0"/>
-    <limit effort="100" velocity="100.0"  lower="0" upper="3.14" />
+    <limit effort="100" velocity="100.0"  lower="-3.14" upper="0" />
   </joint>
   <link name="arm_link_4">
@@ -271,5 +271,5 @@
     </collision>
     <visual name="visual">
-      <origin xyz="-0.05 0 -0.13" rpy="0 0 0"/>
+      <origin xyz="-0.05 0 0.13" rpy="0 0 0"/>
       <geometry>
 	      <box size="0.05 0.05 0.25"/>
@@ -281,5 +281,5 @@
     <parent link="arm_link_4"/>
     <child link="arm_link_5"/>
-    <origin xyz="-0.045 0.0 -0.23" rpy="0 0 3.14"/>
+    <origin xyz="-0.05 0.0 0.23" rpy="0 0 3.14"/>
     <axis xyz="0 1 0" rpy="0 0 0"/>
     <limit effort="100" velocity="100.0"  lower="-1.57" upper="1.57" />
@@ -287,5 +287,5 @@
   <link name="arm_link_5">
     <visual name="visual">
-      <origin xyz="0.0 0 -0.03" rpy="0 0 0"/>
+      <origin xyz="0.0 0 0.03" rpy="0 0 0"/>
       <geometry>
 	      <box size="0.05 0.05 0.08"/>
@@ -297,5 +297,5 @@
     <parent link="arm_link_5"/>
     <child link="arm_link_6"/>
-    <origin xyz="0.0 0.0 -0.06" rpy="0 0 0"/>
+    <origin xyz="0.0 0.0 0.06" rpy="0 0 3.14"/>
     <axis xyz="1 0 0" rpy="0 0 0"/>
     <limit effort="100" velocity="100.0"  lower="-1.57" upper="1.57" />
@@ -303,5 +303,5 @@
   <link name="arm_link_6">
     <visual name="visual">
-      <origin xyz="0.0 0 -0.04" rpy="0 0 0"/>
+      <origin xyz="0.0 0 0.04" rpy="0 0 0"/>
       <geometry>
 	      <box size="0.05 0.03 0.03"/>
